File: pcb/lapis/STM32F405RGT.sch (KiCad schematic (older format))
At the start: 1 part

Commit message: 基板修正途中　ソフト動作確認まで
Parts:
- gave numbers to parts that had none: 1
Changed lines of the file:
@@
 $Descr A4 11693 8268
 encoding utf-8
-Sheet 3 14
+Sheet 2 14
 Title ""
 Date ""
@@
 $EndDescr
 $Comp
-L MCU_ST_STM32F4:STM32F405RGTx U?
+L MCU_ST_STM32F4:STM32F405RGTx U1
 U 1 1 5FA82CA3
 P 5450 3250
-F 0 "U?" H 5450 1361 50  0000 C CNN
+F 0 "U1" H 5450 1361 50  0000 C CNN
 F 1 "STM32F405RGTx" H 5450 1270 50  0000 C CNN
 F 2 "Package_QFP:LQFP-64_10x10mm_P0.5mm" H 4850 1550 50  0001 R CNN
