File: pcb/lapis/power.sch (KiCad schematic (older format))
At the start: 3 parts

Commit message: 基板修正途中　ソフト動作確認まで
Parts:
- removed Q?: Q_PMOS_SGD, symbol Device:Q_PMOS_SGD
- removed SW?: SW_SPDT, symbol Switch:SW_SPDT
- added C14, C19: 0.1u, Capacitor_SMD:C_0201_0603Metric_Pad0.64x0.40mm_HandSolder, symbol Device:C
- added C15: 470p, Capacitor_SMD:C_0201_0603Metric_Pad0.64x0.40mm_HandSolder, symbol Device:C
- added C16: 2.2u, Capacitor_SMD:C_0402_1005Metric_Pad0.74x0.62mm_HandSolder, symbol Device:C
- added D3: LED, LED_SMD:LED_0402_1005Metric_Pad0.77x0.64mm_HandSolder, symbol Device:LED
- added IC4: MIC5219-3.3YM5-TR, SOT95P280X130-5N, symbol lapis-rescue:MIC5219-3.3YM5-TR-SamacSys_Parts
- added J3: Conn_01x02, Connector_Hirose:Hirose_DF13-02P-1.25DSA_1x02_P1.25mm_Vertical, symbol Connector_Generic:Conn_01x02
- added Q5: IRLML6402TRPBF, Package_TO_SOT_SMD:SOT-23, symbol Device:Q_PMOS_GSD
- added R7, R8: 10k, Resistor_SMD:R_0201_0603Metric_Pad0.64x0.40mm_HandSolder, symbol Device:R
- added R9: 1k, Resistor_SMD:R_0201_0603Metric_Pad0.64x0.40mm_HandSolder, symbol Device:R
- added S1: SSSS810701, SSSS810701, symbol SamacSys_Parts:SSSS810701
- R6: renamed from R?; value R -> 10k; footprint (none) -> Resistor_SMD:R_0201_0603Metric_Pad0.64x0.40mm_HandSolder
Connections:
- net labels added: +3.3V, AD_BATT, GND
- wire segments 0 -> 39
- no-connect marks 0 -> 1
Other:
- moved on the sheet: R6
